Commit message: Add parent parameters for the single arms, allow env vars to change the origin of the left & right arms, like we do with the single arms.  Add an intermediate mount joint for the dual-arm configuration

File: warthog_iiwa_description/urdf/warthog_dual_iiwa_14_description.urdf.xacro (robot description, xacro)
@@ -2,20 +2,32 @@
 <robot xmlns:xacro="http://ros.org/wiki/xacro">
   <xacro:arg name="left_prefix" default="left_iiwa_arm" />
-  <xacro:arg name="left_mount" default="left_arm_mount" />
+  <xacro:arg name="left_parent" default="left_arm_mount" />
   <xacro:arg name="left_origin_xyz" default="0 0 0"/>
   <xacro:arg name="left_origin_rpy" default="0 0 0"/>
-  <xacro:arg name="right_mount" default="right_arm_mount" />
+  <xacro:arg name="right_parent" default="right_arm_mount" />
   <xacro:arg name="right_prefix" default="right_iiwa_arm" />
   <xacro:arg name="right_origin_xyz" default="0 0 0"/>
   <xacro:arg name="right_origin_rpy" default="0 0 0"/>
+  <xacro:arg name="hardware_interface" default="PositionJointInterface"/>
   <xacro:include filename="$(find iiwa_description)/urdf/materials.xacro" />
   <xacro:include filename="$(find iiwa_description)/urdf/iiwa14.xacro"/>
-  <xacro:arg name="hardware_interface" default="PositionJointInterface"/>
-  <xacro:arg name="origin_xyz" default="0 0 0"/>
-  <xacro:arg name="origin_rpy" default="0 0 0"/>
-  <xacro:iiwa14 hardware_interface="$(arg hardware_interface)" robot_name="$(arg left_prefix)" parent="$(arg left_mount)">
+  <joint name="$(arg left_prefix)_mount_joint" type="fixed">
+    <parent link="$(arg left_parent)" />
+    <child link="$(arg left_prefix)_mount_link" />
+    <origin xyz="$(optenv WARTHOG_LEFT_IIWA_XYZ 0.0 0.0 0.0)" rpy="$(optenv WARTHOG_LEFT_IIWA_RPY 0 0 0)"/>
+  </joint>
+  <link name="$(arg left_prefix)_mount_link" />
+  <joint name="$(arg right_prefix)_mount_joint" type="fixed">
+    <parent link="$(arg right_parent)" />
+    <child link="$(arg right_prefix)_mount_link" />
+    <origin xyz="$(optenv WARTHOG_RIGHT_IIWA_XYZ 0.0 0.0 0.0)" rpy="$(optenv WARTHOG_RIGHT_IIWA_RPY 0 0 0)"/>
+  </joint>
+  <link name="$(arg right_prefix)_mount_link" />
+  <xacro:iiwa14 hardware_interface="$(arg hardware_interface)" robot_name="$(arg left_prefix)"
+    parent="$(arg left_prefix)_mount_link">
     <origin xyz="$(arg left_origin_xyz)" rpy="$(arg left_origin_rpy)" />
   </xacro:iiwa14>
-  <xacro:iiwa14 hardware_interface="$(arg hardware_interface)" robot_name="$(arg right_prefix)" parent="$(arg right_mount)">
+  <xacro:iiwa14 hardware_interface="$(arg hardware_interface)" robot_name="$(arg right_prefix)"
+    parent="$(arg right_prefix)_mount_link">
     <origin xyz="$(arg right_origin_xyz)" rpy="$(arg right_origin_rpy)" />
   </xacro:iiwa14>

File: warthog_iiwa_description/urdf/warthog_iiwa_14_description.urdf.xacro (robot description, xacro)
@@ -5,13 +5,14 @@
   <xacro:arg name="hardware_interface" default="PositionJointInterface"/>
   <xacro:arg name="robot_name" default="iiwa"/>
+  <xacro:arg name="parent"  default="bulkhead_front_mount_link" />
   <xacro:arg name="origin_xyz" default="0 0 0"/>
   <xacro:arg name="origin_rpy" default="0 0 0"/>
-  <joint name="arm_mount_joint" type="fixed">
-    <parent link="bulkhead_front_mount_link" />
-    <child link="arm_mount_link" />
+  <joint name="$(arg robot_name)_mount_joint" type="fixed">
+    <parent link="$(arg parent)" />
+    <child link="$(arg robot_name)_mount_link" />
     <origin xyz="$(optenv WARTHOG_IIWA_XYZ 0.0 0.0 0.0)" rpy="$(optenv WARTHOG_IIWA_RPY 0 0 0)"/>
   </joint>
-  <link name="arm_mount_link" />
-  <xacro:iiwa14 hardware_interface="$(arg hardware_interface)" robot_name="$(arg robot_name)" parent="arm_mount_link">
+  <link name="$(arg robot_name)_mount_link" />
+  <xacro:iiwa14 hardware_interface="$(arg hardware_interface)" robot_name="$(arg robot_name)" parent="$(arg robot_name)_mount_link">
     <origin xyz="$(arg origin_xyz)" rpy="$(arg origin_rpy)" />
   </xacro:iiwa14>

File: warthog_iiwa_description/urdf/warthog_iiwa_7_description.urdf.xacro (robot description, xacro)
@@ -5,13 +5,14 @@
   <xacro:arg name="hardware_interface" default="PositionJointInterface"/>
   <xacro:arg name="robot_name" default="iiwa"/>
+  <xacro:arg name="parent"  default="bulkhead_front_mount_link" />
   <xacro:arg name="origin_xyz" default="0 0 0"/>
   <xacro:arg name="origin_rpy" default="0 0 0"/>
-  <joint name="arm_mount_joint" type="fixed">
-    <parent link="bulkhead_front_mount_link" />
-    <child link="arm_mount_link" />
+  <joint name="$(arg robot_name)_mount_joint" type="fixed">
+    <parent link="$(arg parent)" />
+    <child link="$(arg robot_name)_mount_link" />
     <origin xyz="$(optenv WARTHOG_IIWA_XYZ 0.0 0.0 0.0)" rpy="$(optenv WARTHOG_IIWA_RPY 0 0 0)"/>
   </joint>
-  <link name="arm_mount_link" />
-  <xacro:iiwa7 hardware_interface="$(arg hardware_interface)" robot_name="$(arg robot_name)" parent="arm_mount_link">
+  <link name="$(arg robot_name)_mount_link" />
+  <xacro:iiwa7 hardware_interface="$(arg hardware_interface)" robot_name="$(arg robot_name)" parent="$(arg robot_name)_mount_link">
     <origin xyz="$(arg origin_xyz)" rpy="$(arg origin_rpy)" />
   </xacro:iiwa7>
