Commit message: Update UR arm packages (as per husky_manipulation)

File: warthog_ur_description/urdf/warthog_dual_ur10_description.urdf.xacro (robot description, xacro)
@@ -1,18 +1,16 @@
+<?xml version="1.0"?>
 <robot xmlns:xacro="http://ros.org/wiki/xacro">
-  <xacro:include filename="$(find ur_description)/urdf/ur10.urdf.xacro" />
-  <xacro:arg name="kinematics_config" default="$(find ur_description)/config/ur10_default.yaml" />
-  <xacro:arg name="transmission_hw_interface" default="hardware_interface/PositionJointInterface"/>
-  <xacro:include filename="$(find ur_description)/urdf/common.gazebo.xacro" />
+  <xacro:include filename="$(find ur_description)/urdf/inc/ur10_macro.xacro" />
   <joint name="left_arm_mount_joint" type="fixed">
-    <parent link="bulkhead_front_mount_link" />
+    <parent link="left_arm_bulkhead_link" />
     <child link="left_ur_arm_base_link" />
-    <origin xyz="$(optenv WARTHOG_LEFT_UR_XYZ 0.0 0.2 0.0)" rpy="$(optenv WARTHOG_LEFT_UR_RPY 0 0 3.14159)"/>
+    <origin xyz="$(optenv WARTHOG_LEFT_UR_XYZ 0 0 0)" rpy="$(optenv WARTHOG_LEFT_UR_RPY 0 0 0)"/>
   </joint>
   <joint name="right_arm_mount_joint" type="fixed">
-    <parent link="bulkhead_front_mount_link" />
+    <parent link="right_arm_bulkhead_link" />
     <child link="right_ur_arm_base_link" />
-    <origin xyz="$(optenv WARTHOG_RIGHT_UR_XYZ 0.0 -0.2 0.0)" rpy="$(optenv WARTHOG_RIGHT_UR_RPY 0 0 3.14159)"/>
+    <origin xyz="$(optenv WARTHOG_RIGHT_UR_XYZ 0 0 0)" rpy="$(optenv WARTHOG_RIGHT_UR_RPY 0 0 0)"/>
   </joint>
-  <xacro:ur10_robot prefix="left_ur_arm_" joint_limited="true" kinematics_file="${load_yaml('$(arg kinematics_config)')}" />
-  <xacro:ur10_robot prefix="right_ur_arm_" joint_limited="true" kinematics_file="${load_yaml('$(arg kinematics_config)')}" />
+  <xacro:ur10_robot prefix="right_ur_arm_" />
+  <xacro:ur10_robot prefix="left_ur_arm_" />
 </robot>

File: warthog_ur_description/urdf/warthog_dual_ur10_e_description.urdf.xacro (robot description, xacro)
@@ -1,18 +1,16 @@
+<?xml version="1.0"?>
 <robot xmlns:xacro="http://ros.org/wiki/xacro">
-  <xacro:include filename="$(find ur_e_description)/urdf/ur10e.urdf.xacro" />
-  <xacro:arg name="kinematics_config" default="$(find ur_e_description)/config/ur10e_default.yaml" />
-  <xacro:arg name="transmission_hw_interface" default="hardware_interface/PositionJointInterface"/>
-  <xacro:include filename="$(find ur_e_description)/urdf/common.gazebo.xacro" />
+  <xacro:include filename="$(find ur_description)/urdf/inc/ur10e_macro.xacro" />
   <joint name="left_arm_mount_joint" type="fixed">
-    <parent link="bulkhead_front_mount_link" />
+    <parent link="left_arm_bulkhead_link" />
     <child link="left_ur_arm_base_link" />
-    <origin xyz="$(optenv WARTHOG_LEFT_UR_XYZ 0.0 0.2 0.0)" rpy="$(optenv WARTHOG_LEFT_UR_RPY 0 0 3.14159)"/>
+    <origin xyz="$(optenv WARTHOG_LEFT_UR_XYZ 0 0 0)" rpy="$(optenv WARTHOG_LEFT_UR_RPY 0 0 0)"/>
   </joint>
   <joint name="right_arm_mount_joint" type="fixed">
-    <parent link="bulkhead_front_mount_link" />
+    <parent link="right_arm_bulkhead_link" />
     <child link="right_ur_arm_base_link" />
-    <origin xyz="$(optenv WARTHOG_RIGHT_UR_XYZ 0.0 -0.2 0.0)" rpy="$(optenv WARTHOG_RIGHT_UR_RPY 0 0 3.14159)"/>
+    <origin xyz="$(optenv WARTHOG_RIGHT_UR_XYZ 0 0 0)" rpy="$(optenv WARTHOG_RIGHT_UR_RPY 0 0 0)"/>
   </joint>
-  <xacro:ur10e_robot prefix="left_ur_arm_" joint_limited="true" kinematics_file="${load_yaml('$(arg kinematics_config)')}" />
-  <xacro:ur10e_robot prefix="right_ur_arm_" joint_limited="true" kinematics_file="${load_yaml('$(arg kinematics_config)')}" />
+  <xacro:ur10e_robot prefix="right_ur_arm_" />
+  <xacro:ur10e_robot prefix="left_ur_arm_" />
 </robot>

File: warthog_ur_description/urdf/warthog_dual_ur5_description.urdf.xacro (robot description, xacro)
@@ -1,18 +1,16 @@
+<?xml version="1.0"?>
 <robot xmlns:xacro="http://ros.org/wiki/xacro">
-  <xacro:include filename="$(find ur_description)/urdf/ur5.urdf.xacro" />
-  <xacro:arg name="kinematics_config" default="$(find ur_description)/config/ur5_default.yaml" />
-  <xacro:arg name="transmission_hw_interface" default="hardware_interface/PositionJointInterface"/>
-  <xacro:include filename="$(find ur_description)/urdf/common.gazebo.xacro" />
+  <xacro:include filename="$(find ur_description)/urdf/inc/ur5_macro.xacro" />
   <joint name="left_arm_mount_joint" type="fixed">
-    <parent link="bulkhead_front_mount_link" />
+    <parent link="left_arm_bulkhead_link" />
     <child link="left_ur_arm_base_link" />
-    <origin xyz="$(optenv WARTHOG_LEFT_UR_XYZ 0.0 0.2 0.0)" rpy="$(optenv WARTHOG_LEFT_UR_RPY 0 0 3.14159)"/>
+    <origin xyz="$(optenv WARTHOG_LEFT_UR_XYZ 0 0 0)" rpy="$(optenv WARTHOG_LEFT_UR_RPY 0 0 0)"/>
   </joint>
   <joint name="right_arm_mount_joint" type="fixed">
-    <parent link="bulkhead_front_mount_link" />
+    <parent link="right_arm_bulkhead_link" />
     <child link="right_ur_arm_base_link" />
-    <origin xyz="$(optenv WARTHOG_RIGHT_UR_XYZ 0.0 -0.2 0.0)" rpy="$(optenv WARTHOG_RIGHT_UR_RPY 0 0 3.14159)"/>
+    <origin xyz="$(optenv WARTHOG_RIGHT_UR_XYZ 0 0 0)" rpy="$(optenv WARTHOG_RIGHT_UR_RPY 0 0 0)"/>
   </joint>
-  <xacro:ur5_robot prefix="left_ur_arm_" joint_limited="true" kinematics_file="${load_yaml('$(arg kinematics_config)')}" />
-  <xacro:ur5_robot prefix="right_ur_arm_" joint_limited="true" kinematics_file="${load_yaml('$(arg kinematics_config)')}" />
+  <xacro:ur5_robot prefix="right_ur_arm_" />
+  <xacro:ur5_robot prefix="left_ur_arm_" />
 </robot>

File: warthog_ur_description/urdf/warthog_dual_ur5_e_description.urdf.xacro (robot description, xacro)
@@ -1,18 +1,16 @@
+<?xml version="1.0"?>
 <robot xmlns:xacro="http://ros.org/wiki/xacro">
-  <xacro:include filename="$(find ur_e_description)/urdf/ur5e.urdf.xacro" />
-  <xacro:arg name="kinematics_config" default="$(find ur_e_description)/config/ur5e_default.yaml" />
-  <xacro:arg name="transmission_hw_interface" default="hardware_interface/PositionJointInterface"/>
-  <xacro:include filename="$(find ur_e_description)/urdf/common.gazebo.xacro" />
+  <xacro:include filename="$(find ur_description)/urdf/inc/ur5e_macro.xacro" />
   <joint name="left_arm_mount_joint" type="fixed">
-    <parent link="bulkhead_front_mount_link" />
+    <parent link="left_arm_bulkhead_link" />
     <child link="left_ur_arm_base_link" />
-    <origin xyz="$(optenv WARTHOG_LEFT_UR_XYZ 0.0 0.2 0.0)" rpy="$(optenv WARTHOG_LEFT_UR_RPY 0 0 3.14159)"/>
+    <origin xyz="$(optenv WARTHOG_LEFT_UR_XYZ 0 0 0)" rpy="$(optenv WARTHOG_LEFT_UR_RPY 0 0 0)"/>
   </joint>
   <joint name="right_arm_mount_joint" type="fixed">
-    <parent link="bulkhead_front_mount_link" />
+    <parent link="right_arm_bulkhead_link" />
     <child link="right_ur_arm_base_link" />
-    <origin xyz="$(optenv WARTHOG_RIGHT_UR_XYZ 0.0 -0.2 0.0)" rpy="$(optenv WARTHOG_RIGHT_UR_RPY 0 0 3.14159)"/>
+    <origin xyz="$(optenv WARTHOG_RIGHT_UR_XYZ 0 0 0)" rpy="$(optenv WARTHOG_RIGHT_UR_RPY 0 0 0)"/>
   </joint>
-  <xacro:ur5e_robot prefix="left_ur_arm_" joint_limited="true" kinematics_file="${load_yaml('$(arg kinematics_config)')}" />
-  <xacro:ur5e_robot prefix="right_ur_arm_" joint_limited="true" kinematics_file="${load_yaml('$(arg kinematics_config)')}" />
+  <xacro:ur5e_robot prefix="right_ur_arm_" />
+  <xacro:ur5e_robot prefix="left_ur_arm_" />
 </robot>

File: warthog_ur_description/urdf/warthog_ur10_description.urdf.xacro (robot description, xacro)
@@ -1,12 +1,10 @@
+<?xml version="1.0"?>
 <robot xmlns:xacro="http://ros.org/wiki/xacro">
-  <xacro:include filename="$(find ur_description)/urdf/ur10.urdf.xacro" />
-  <xacro:arg name="kinematics_config" default="$(find ur_description)/config/ur10_default.yaml" />
-  <xacro:arg name="transmission_hw_interface" default="hardware_interface/PositionJointInterface"/>
-  <xacro:include filename="$(find ur_description)/urdf/common.gazebo.xacro" />
+  <xacro:include filename="$(find ur_description)/urdf/inc/ur10_macro.xacro" />
   <joint name="arm_mount_joint" type="fixed">
-    <parent link="bulkhead_front_mount_link" />
+    <parent link="top_plate_front_link" />
     <child link="ur_arm_base_link" />
-    <origin xyz="$(optenv WARTHOG_UR_XYZ 0.0 0.0 0.0)" rpy="$(optenv WARTHOG_UR_RPY 0 0 3.1415927)"/>
+    <origin xyz="$(optenv WARTHOG_UR_XYZ -0.105 0.0 0.0)" rpy="$(optenv WARTHOG_UR_RPY 0 0 3.1415927)"/>
   </joint>
-  <xacro:ur10_robot prefix="ur_arm_" joint_limited="true" kinematics_file="${load_yaml('$(arg kinematics_config)')}" />
+  <xacro:ur10_robot prefix="ur_arm_" />
 </robot>

File: warthog_ur_description/urdf/warthog_ur10_e_description.urdf.xacro (robot description, xacro)
@@ -1,12 +1,10 @@
+<?xml version="1.0"?>
 <robot xmlns:xacro="http://ros.org/wiki/xacro">
-  <xacro:include filename="$(find ur_e_description)/urdf/ur10e.urdf.xacro" />
-  <xacro:arg name="kinematics_config" default="$(find ur_e_description)/config/ur10e_default.yaml" />
-  <xacro:arg name="transmission_hw_interface" default="hardware_interface/PositionJointInterface"/>
-  <xacro:include filename="$(find ur_e_description)/urdf/common.gazebo.xacro" />
+  <xacro:include filename="$(find ur_description)/urdf/inc/ur10e_macro.xacro" />
   <joint name="arm_mount_joint" type="fixed">
-    <parent link="bulkhead_front_mount_link" />
+    <parent link="top_plate_front_link" />
     <child link="ur_arm_base_link" />
-    <origin xyz="$(optenv WARTHOG_UR_XYZ 0.0 0.0 0.0)" rpy="$(optenv WARTHOG_UR_RPY 0 0 3.1415927)"/>
+    <origin xyz="$(optenv WARTHOG_UR_XYZ -0.105 0.0 0.0)" rpy="$(optenv WARTHOG_UR_RPY 0 0 3.1415927)"/>
   </joint>
-  <xacro:ur10e_robot prefix="ur_arm_" joint_limited="true" kinematics_file="${load_yaml('$(arg kinematics_config)')}" />
+  <xacro:ur10e_robot prefix="ur_arm_" />
 </robot>

File: warthog_ur_description/urdf/warthog_ur5_description.urdf.xacro (robot description, xacro)
@@ -1,12 +1,10 @@
+<?xml version="1.0"?>
 <robot xmlns:xacro="http://ros.org/wiki/xacro">
-  <xacro:include filename="$(find ur_description)/urdf/ur5.urdf.xacro" />
-  <xacro:arg name="kinematics_config" default="$(find ur_description)/config/ur5_default.yaml" />
-  <xacro:arg name="transmission_hw_interface" default="hardware_interface/PositionJointInterface"/>
-  <xacro:include filename="$(find ur_description)/urdf/common.gazebo.xacro" />
+  <xacro:include filename="$(find ur_description)/urdf/inc/ur5_macro.xacro" />
   <joint name="arm_mount_joint" type="fixed">
-    <parent link="bulkhead_front_mount_link" />
+    <parent link="top_plate_front_link" />
     <child link="ur_arm_base_link" />
-    <origin xyz="$(optenv WARTHOG_UR_XYZ 0.0 0.0 0.0)" rpy="$(optenv WARTHOG_UR_RPY 0 0 3.1415927)"/>
+    <origin xyz="$(optenv WARTHOG_UR_XYZ -0.105 0.0 0.0)" rpy="$(optenv WARTHOG_UR_RPY 0 0 3.1415927)"/>
   </joint>
-  <xacro:ur5_robot prefix="ur_arm_" joint_limited="true" kinematics_file="${load_yaml('$(arg kinematics_config)')}" />
+  <xacro:ur5_robot prefix="ur_arm_" />
 </robot>

File: warthog_ur_description/urdf/warthog_ur5_e_description.urdf.xacro (robot description, xacro)
@@ -1,12 +1,10 @@
+<?xml version="1.0"?>
 <robot xmlns:xacro="http://ros.org/wiki/xacro">
-  <xacro:include filename="$(find ur_e_description)/urdf/ur5e.urdf.xacro" />
-  <xacro:arg name="kinematics_config" default="$(find ur_e_description)/config/ur5e_default.yaml" />
-  <xacro:arg name="transmission_hw_interface" default="hardware_interface/PositionJointInterface"/>
-  <xacro:include filename="$(find ur_e_description)/urdf/common.gazebo.xacro" />
+  <xacro:include filename="$(find ur_description)/urdf/inc/ur5e_macro.xacro" />
   <joint name="arm_mount_joint" type="fixed">
-    <parent link="bulkhead_front_mount_link" />
+    <parent link="top_plate_front_link" />
     <child link="ur_arm_base_link" />
-    <origin xyz="$(optenv WARTHOG_UR_XYZ 0.0 0.0 0.0)" rpy="$(optenv WARTHOG_UR_RPY 0 0 3.1415927)"/>
+    <origin xyz="$(optenv WARTHOG_UR_XYZ -0.105 0.0 0.0)" rpy="$(optenv WARTHOG_UR_RPY 0 0 3.1415927)"/>
   </joint>
-  <xacro:ur5e_robot prefix="ur_arm_" joint_limited="true" kinematics_file="${load_yaml('$(arg kinematics_config)')}" />
+  <xacro:ur5e_robot prefix="ur_arm_" />
 </robot>
