Commit message: Change top_plate_front_link to top_chassis_link

File: warthog_ur_description/urdf/warthog_ur10_description.urdf.xacro (robot description, xacro)
@@ -3,5 +3,5 @@
   <xacro:include filename="$(find ur_description)/urdf/inc/ur10_macro.xacro" />
   <joint name="arm_mount_joint" type="fixed">
-    <parent link="top_plate_front_link" />
+    <parent link="top_chassis_link" />
     <child link="ur_arm_base_link" />
     <origin xyz="$(optenv WARTHOG_UR_XYZ -0.105 0.0 0.0)" rpy="$(optenv WARTHOG_UR_RPY 0 0 3.1415927)"/>

File: warthog_ur_description/urdf/warthog_ur10_e_description.urdf.xacro (robot description, xacro)
@@ -3,5 +3,5 @@
   <xacro:include filename="$(find ur_description)/urdf/inc/ur10e_macro.xacro" />
   <joint name="arm_mount_joint" type="fixed">
-    <parent link="top_plate_front_link" />
+    <parent link="top_chassis_link" />
     <child link="ur_arm_base_link" />
     <origin xyz="$(optenv WARTHOG_UR_XYZ -0.105 0.0 0.0)" rpy="$(optenv WARTHOG_UR_RPY 0 0 3.1415927)"/>

File: warthog_ur_description/urdf/warthog_ur5_description.urdf.xacro (robot description, xacro)
@@ -3,5 +3,5 @@
   <xacro:include filename="$(find ur_description)/urdf/inc/ur5_macro.xacro" />
   <joint name="arm_mount_joint" type="fixed">
-    <parent link="top_plate_front_link" />
+    <parent link="top_chassis_link" />
     <child link="ur_arm_base_link" />
     <origin xyz="$(optenv WARTHOG_UR_XYZ -0.105 0.0 0.0)" rpy="$(optenv WARTHOG_UR_RPY 0 0 3.1415927)"/>

File: warthog_ur_description/urdf/warthog_ur5_e_description.urdf.xacro (robot description, xacro)
@@ -3,5 +3,5 @@
   <xacro:include filename="$(find ur_description)/urdf/inc/ur5e_macro.xacro" />
   <joint name="arm_mount_joint" type="fixed">
-    <parent link="top_plate_front_link" />
+    <parent link="top_chassis_link" />
     <child link="ur_arm_base_link" />
     <origin xyz="$(optenv WARTHOG_UR_XYZ -0.105 0.0 0.0)" rpy="$(optenv WARTHOG_UR_RPY 0 0 3.1415927)"/>

Commit message: Change default position and orientation of arm

File: warthog_ur_description/urdf/warthog_ur10_description.urdf.xacro (robot description, xacro)
@@ -5,5 +5,5 @@
     <parent link="top_chassis_link" />
     <child link="ur_arm_base_link" />
-    <origin xyz="$(optenv WARTHOG_UR_XYZ -0.105 0.0 0.0)" rpy="$(optenv WARTHOG_UR_RPY 0 0 3.1415927)"/>
+    <origin xyz="$(optenv WARTHOG_UR_XYZ 0.3 0 0)" rpy="$(optenv WARTHOG_UR_RPY 0 0 0)"/>
   </joint>
   <xacro:ur10_robot prefix="ur_arm_" />

File: warthog_ur_description/urdf/warthog_ur10_e_description.urdf.xacro (robot description, xacro)
@@ -5,5 +5,5 @@
     <parent link="top_chassis_link" />
     <child link="ur_arm_base_link" />
-    <origin xyz="$(optenv WARTHOG_UR_XYZ -0.105 0.0 0.0)" rpy="$(optenv WARTHOG_UR_RPY 0 0 3.1415927)"/>
+    <origin xyz="$(optenv WARTHOG_UR_XYZ 0.3 0 0)" rpy="$(optenv WARTHOG_UR_RPY 0 0 0)"/>
   </joint>
   <xacro:ur10e_robot prefix="ur_arm_" />

File: warthog_ur_description/urdf/warthog_ur5_description.urdf.xacro (robot description, xacro)
@@ -5,5 +5,5 @@
     <parent link="top_chassis_link" />
     <child link="ur_arm_base_link" />
-    <origin xyz="$(optenv WARTHOG_UR_XYZ -0.105 0.0 0.0)" rpy="$(optenv WARTHOG_UR_RPY 0 0 3.1415927)"/>
+    <origin xyz="$(optenv WARTHOG_UR_XYZ 0.3 0 0)" rpy="$(optenv WARTHOG_UR_RPY 0 0 0)"/>
   </joint>
   <xacro:ur5_robot prefix="ur_arm_" />

File: warthog_ur_description/urdf/warthog_ur5_e_description.urdf.xacro (robot description, xacro)
@@ -5,5 +5,5 @@
     <parent link="top_chassis_link" />
     <child link="ur_arm_base_link" />
-    <origin xyz="$(optenv WARTHOG_UR_XYZ -0.105 0.0 0.0)" rpy="$(optenv WARTHOG_UR_RPY 0 0 3.1415927)"/>
+    <origin xyz="$(optenv WARTHOG_UR_XYZ 0.3 0 0)" rpy="$(optenv WARTHOG_UR_RPY 0 0 0)"/>
   </joint>
   <xacro:ur5e_robot prefix="ur_arm_" />

Commit message: Move default XYZ to origin of top_chassis_link

File: warthog_ur_description/urdf/warthog_ur10_description.urdf.xacro (robot description, xacro)
@@ -5,5 +5,5 @@
     <parent link="top_chassis_link" />
     <child link="ur_arm_base_link" />
-    <origin xyz="$(optenv WARTHOG_UR_XYZ 0.3 0 0)" rpy="$(optenv WARTHOG_UR_RPY 0 0 0)"/>
+    <origin xyz="$(optenv WARTHOG_UR_XYZ 0 0 0)" rpy="$(optenv WARTHOG_UR_RPY 0 0 0)"/>
   </joint>
   <xacro:ur10_robot prefix="ur_arm_" />

File: warthog_ur_description/urdf/warthog_ur10_e_description.urdf.xacro (robot description, xacro)
@@ -5,5 +5,5 @@
     <parent link="top_chassis_link" />
     <child link="ur_arm_base_link" />
-    <origin xyz="$(optenv WARTHOG_UR_XYZ 0.3 0 0)" rpy="$(optenv WARTHOG_UR_RPY 0 0 0)"/>
+    <origin xyz="$(optenv WARTHOG_UR_XYZ 0 0 0)" rpy="$(optenv WARTHOG_UR_RPY 0 0 0)"/>
   </joint>
   <xacro:ur10e_robot prefix="ur_arm_" />

File: warthog_ur_description/urdf/warthog_ur5_description.urdf.xacro (robot description, xacro)
@@ -5,5 +5,5 @@
     <parent link="top_chassis_link" />
     <child link="ur_arm_base_link" />
-    <origin xyz="$(optenv WARTHOG_UR_XYZ 0.3 0 0)" rpy="$(optenv WARTHOG_UR_RPY 0 0 0)"/>
+    <origin xyz="$(optenv WARTHOG_UR_XYZ 0 0 0)" rpy="$(optenv WARTHOG_UR_RPY 0 0 0)"/>
   </joint>
   <xacro:ur5_robot prefix="ur_arm_" />

File: warthog_ur_description/urdf/warthog_ur5_e_description.urdf.xacro (robot description, xacro)
@@ -5,5 +5,5 @@
     <parent link="top_chassis_link" />
     <child link="ur_arm_base_link" />
-    <origin xyz="$(optenv WARTHOG_UR_XYZ 0.3 0 0)" rpy="$(optenv WARTHOG_UR_RPY 0 0 0)"/>
+    <origin xyz="$(optenv WARTHOG_UR_XYZ 0 0 0)" rpy="$(optenv WARTHOG_UR_RPY 0 0 0)"/>
   </joint>
   <xacro:ur5e_robot prefix="ur_arm_" />
